File: DimmerV1.2.brd (EAGLE design)
At the start: 53.5 x 56 mm, 21 parts, among them J1 AC IN, J2 SWITCH, J3 ICSP, T1 2N6073AG, U1 HLK-PM03, U3 NRF24L01, U4 ATMEGA328P_TQFP

Commit message: Board layout fixes (C1)
Parts:
- moved C1 2.00 mm to (16.0, 9.20)
Changed lines of the file:
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@@
 </autorouter>
 <elements>
-<element name="C1" library="SparkFun-Capacitors" package="0805" value="0.1uF" x="14" y="9.2" rot="R270"/>
+<element name="C1" library="SparkFun-Capacitors" package="0805" value="0.1uF" x="16" y="9.2" rot="R270"/>
 <element name="J1" library="SparkFun-Connectors" package="SCREWTERMINAL-5MM-3" value="AC IN" x="15.5" y="53" rot="R180">
 <attribute name="STOREFRONT_ID" value="PRT-08433" x="15.5" y="53" size="1.778" layer="27" rot="R180" display="off"/>
@@
 <wire x1="19.2074" y1="9.9" x2="20.5" y2="9.9" width="0.254" layer="1"/>
 <wire x1="20.5" y1="9.9" x2="20.5" y2="8.3" width="0.254" layer="1"/>
-<wire x1="14" y1="8.3" x2="19.2074" y2="8.3" width="0.254" layer="1"/>
+<wire x1="16" y1="8.3" x2="19.2074" y2="8.3" width="0.254" layer="1"/>
+<wire x1="16" y1="8.3" x2="14" y2="8.3" width="0.254" layer="1"/>
 <wire x1="14" y1="8.3" x2="12.13" y2="6.43" width="0.254" layer="1"/>
 <wire x1="12.13" y1="6.43" x2="2.95" y2="6.43" width="0.254" layer="1"/>
